File: clavier/clavier.sch (KiCad schematic (older format))
At the start: 7 parts

Commit message: added TODO, updated clavier
Parts:
- added LED_maj, LED_num, LED_spé: LED, symbol LED
- added R_led (x3), R_usb (x2): R, symbol R
- C: renamed from C?; value C_Small -> 4.7µF
- C: renamed from C?; value C_Small -> 10µF
- L: renamed from L?; value L_Small -> 10µH
- gave numbers to parts that had none: 3
Connections:
- wire segments 74 -> 95
Other:
- moved on the sheet: Flash_memory
Changed lines of the file:
@@
 $EndDescr
 $Comp
-L ATXMEGA16A4U-AU U?
+L ATXMEGA16A4U-AU µP
 U 1 1 5E14C77C
 P 4700 3600
-F 0 "U?" H 3950 4800 50  0000 L BNN
+F 0 "µP" H 3950 4800 50  0000 L BNN
 F 1 "ATXMEGA16A4U-AU" H 5050 2350 50  0000 L BNN
 F 2 "TQFP44" H 4700 3600 50  0001 C CIN
@@
 VCC
 $Comp
-L LM3670 U?
+L LM3670 Alim
 U 1 1 5E14E048
 P 2800 3150
-F 0 "U?" H 2800 3150 60  0000 C CNN
+F 0 "Alim" H 2800 3300 60  0000 C CNN
 F 1 "LM3670" H 2800 3150 60  0000 C CNN
 F 2 "" H 2800 3150 60  0001 C CNN
@@
 $EndComp
 $Comp
-L C_Small C?
+L C_Small C
 U 1 1 5E14E10B
 P 2800 3650
-F 0 "C?" H 2810 3720 50  0000 L CNN
-F 1 "C_Small" H 2810 3570 50  0000 L CNN
+F 0 "C" H 2810 3720 50  0000 L CNN
+F 1 "4.7µF" H 2810 3570 50  0000 L CNN
 F 2 "" H 2800 3650 50  0001 C CNN
 F 3 "" H 2800 3650 50  0001 C CNN
@@
 $EndComp
 $Comp
-L L_Small L?
+L L_Small L
 U 1 1 5E14E2A2
 P 2700 2750
-F 0 "L?" H 2730 2790 50  0000 L CNN
-F 1 "L_Small" H 2730 2710 50  0000 L CNN
+F 0 "L" H 2730 2790 50  0000 L CNN
+F 1 "10µH" H 2730 2710 50  0000 L CNN
 F 2 "" H 2700 2750 50  0001 C CNN
 F 3 "" H 2700 2750 50  0001 C CNN
@@
 VCC
 $Comp
-L C_Small C?
+L C_Small C
 U 1 1 5E14E3E8
 P 3100 2650
-F 0 "C?" H 3110 2720 50  0000 L CNN
-F 1 "C_Small" H 3110 2570 50  0000 L CNN
+F 0 "C" H 3110 2720 50  0000 L CNN
+F 1 "10µF" H 3110 2570 50  0000 L CNN
 F 2 "" H 3100 2650 50  0001 C CNN
 F 3 "" H 3100 2650 50  0001 C CNN
@@
 $EndComp
 $Comp
-L MX25R6435F-SOP U?
+L MX25R6435F-SOP Flash_memory
 U 1 1 5E1504AF
-P 6650 4500
-F 0 "U?" V 6200 4500 60  0000 C CNN
-F 1 "MX25R6435F-SOP" V 6100 4500 60  0000 C CNN
-F 2 "" H 7000 4500 60  0001 C CNN
-F 3 "" H 7000 4500 60  0001 C CNN
-	1    6650 4500
+P 7550 4500
+F 0 "Flash_memory" V 7200 4500 60  0000 C CNN
+F 1 "MX25R6435F-SOP" V 7000 4500 60  0000 C CNN
+F 2 "" H 7900 4500 60  0001 C CNN
+F 3 "" H 7900 4500 60  0001 C CNN
+	1    7550 4500
 	0    1    1    0
 $EndComp
@@
 L GNDREF #PWR?
 U 1 1 5E150615
-P 5950 4950
-F 0 "#PWR?" H 5950 4700 50  0001 C CNN
-F 1 "GNDREF" H 5950 4800 50  0000 C CNN
-F 2 "" H 5950 4950 50  0001 C CNN
-F 3 "" H 5950 4950 50  0001 C CNN
-	1    5950 4950
-	1    0    0    -1
-$EndComp
-Text GLabel 7350 4050 2    60   Output ~ 0
+P 6850 4950
+F 0 "#PWR?" H 6850 4700 50  0001 C CNN
+F 1 "GNDREF" H 6850 4800 50  0000 C CNN
+F 2 "" H 6850 4950 50  0001 C CNN
+F 3 "" H 6850 4950 50  0001 C CNN
+	1    6850 4950
+	1    0    0    -1
+$EndComp
+Text GLabel 8250 4050 2    60   Output ~ 0
 VCC
 Entry Wire Line
@@
 	0    1    1    0
 $EndComp
+$Comp
+L R R_usb
+U 1 1 5E28492F
+P 3200 4500
+F 0 "R_usb" V 3280 4500 50  0000 C CNN
+F 1 "R" V 3200 4500 50  0000 C CNN
+F 2 "" V 3130 4500 50  0001 C CNN
+F 3 "" H 3200 4500 50  0001 C CNN
+	1    3200 4500
+	0    1    1    0
+$EndComp
+$Comp
+L R R_usb
+U 1 1 5E28496A
+P 3500 4600
+F 0 "R_usb" V 3580 4600 50  0000 C CNN
+F 1 "R" V 3500 4600 50  0000 C CNN
+F 2 "" V 3430 4600 50  0001 C CNN
+F 3 "" H 3500 4600 50  0001 C CNN
+	1    3500 4600
+	0    1    1    0
+$EndComp
+$Comp
+L LED LED_spé
+U 1 1 5E2852E9
+P 8050 2650
+F 0 "LED_spé" H 8050 2750 50  0000 C CNN
+F 1 "LED" H 8050 2550 50  0000 C CNN
+F 2 "" H 8050 2650 50  0001 C CNN
+F 3 "" H 8050 2650 50  0001 C CNN
+	1    8050 2650
+	0    1    1    0
+$EndComp
+$Comp
+L LED LED_num
+U 1 1 5E28533E
+P 7050 2650
+F 0 "LED_num" H 7050 2750 50  0000 C CNN
+F 1 "LED" H 7050 2550 50  0000 C CNN
+F 2 "" H 7050 2650 50  0001 C CNN
+F 3 "" H 7050 2650 50  0001 C CNN
+	1    7050 2650
+	0    1    1    0
+$EndComp
+$Comp
+L LED LED_maj
+U 1 1 5E28538E
+P 7550 2650
+F 0 "LED_maj" H 7550 2750 50  0000 C CNN
+F 1 "LED" H 7550 2550 50  0000 C CNN
+F 2 "" H 7550 2650 50  0001 C CNN
+F 3 "" H 7550 2650 50  0001 C CNN
+	1    7550 2650
+	0    1    1    0
+$EndComp
+$Comp
+L GNDREF #PWR?
+U 1 1 5E28567D
+P 7550 2800
+F 0 "#PWR?" H 7550 2550 50  0001 C CNN
+F 1 "GNDREF" H 7550 2650 50  0000 C CNN
+F 2 "" H 7550 2800 50  0001 C CNN
+F 3 "" H 7550 2800 50  0001 C CNN
+	1    7550 2800
+	1    0    0    -1
+$EndComp
 Wire Wire Line
 	4550 4900 4650 4900
@@
 Connection ~ 3000 2650
 Wire Wire Line
-	5950 4050 6000 4050
-Wire Wire Line
-	6000 4050 6000 4950
-Wire Wire Line
-	6000 4950 5950 4950
-Wire Wire Line
-	5900 4500 5600 4500
+	6850 4050 6900 4050
+Wire Wire Line
+	6900 4050 6900 4950
+Wire Wire Line
+	6900 4950 6850 4950
+Wire Wire Line
+	5600 4500 6750 4500
 Wire Wire Line
 	5600 4600 5850 5400
 Wire Wire Line
-	5850 5400 7450 5400
-Wire Wire Line
-	7450 5400 7450 4650
-Wire Wire Line
-	7450 4650 7350 4650
-Wire Wire Line
-	7350 4950 7350 5350
-Wire Wire Line
-	7350 5350 5900 5350
+	5850 5400 8350 5400
+Wire Wire Line
+	8350 5400 8350 4650
+Wire Wire Line
+	8350 4650 8250 4650
+Wire Wire Line
+	8250 5350 8250 4950
+Wire Wire Line
+	5900 5350 8250 5350
 Wire Wire Line
 	5900 5350 5600 4400
@@
 	6250 1750 6250 2050
 Wire Wire Line
-	3800 4500 2950 4500
-Wire Wire Line
-	3800 4600 2950 4600
+	3800 4500 3350 4500
+Wire Wire Line
+	3050 4500 2950 4500
+Wire Wire Line
+	3800 4600 3650 4600
+Wire Wire Line
+	3350 4600 2950 4600
 Wire Wire Line
 	2550 4900 2650 4900
@@
 Wire Wire Line
 	2800 3750 2800 3850
-Wire Wire Line
-	5900 4500 5950 4350
 Wire Bus Line
 	6250 2250 6250 3550
 Wire Bus Line
 	6250 3550 5900 3550
+Wire Wire Line
+	6750 4350 6850 4350
+Wire Wire Line
+	6750 4500 6750 4350
+Wire Wire Line
+	7050 2800 7550 2800
+Wire Wire Line
+	7550 2800 8050 2800
+Connection ~ 7550 2800
+Wire Wire Line
+	5600 4300 5800 4300
+Wire Wire Line
+	5800 4300 5800 4400
+Wire Wire Line
+	5800 4400 6550 4400
+Wire Wire Line
+	6550 4400 6550 2500
+Wire Wire Line
+	6550 2500 6650 2500
+Wire Wire Line
+	6950 2500 7050 2500
+Wire Wire Line
+	3800 3200 3750 3200
+Wire Wire Line
+	3750 3200 3750 1500
+Wire Wire Line
+	3750 1500 7550 1500
+Wire Wire Line
+	7550 1500 7550 2100
+Wire Wire Line
+	7550 2400 7550 2500
+Wire Wire Line
+	3800 3300 3650 3300
+Wire Wire Line
+	3650 3300 3650 1400
+Wire Wire Line
+	3650 1400 8050 1400
+Wire Wire Line
+	8050 1400 8050 2100
+Wire Wire Line
+	8050 2400 8050 2500
+$Comp
+L R R_led
+U 1 1 5E285984
+P 6800 2500
+F 0 "R_led" V 6880 2500 50  0000 C CNN
+F 1 "R" V 6800 2500 50  0000 C CNN
+F 2 "" V 6730 2500 50  0001 C CNN
+F 3 "" H 6800 2500 50  0001 C CNN
+	1    6800 2500
+	0    1    1    0
+$EndComp
+$Comp
+L R R_led
+U 1 1 5E285A19
+P 7550 2250
+F 0 "R_led" V 7630 2250 50  0000 C CNN
+F 1 "R" V 7550 2250 50  0000 C CNN
+F 2 "" V 7480 2250 50  0001 C CNN
+F 3 "" H 7550 2250 50  0001 C CNN
+	1    7550 2250
+	1    0    0    -1
+$EndComp
+$Comp
+L R R_led
+U 1 1 5E285A78
+P 8050 2250
+F 0 "R_led" V 8130 2250 50  0000 C CNN
+F 1 "R" V 8050 2250 50  0000 C CNN
+F 2 "" V 7980 2250 50  0001 C CNN
+F 3 "" H 8050 2250 50  0001 C CNN
+	1    8050 2250
+	1    0    0    -1
+$EndComp
 $EndSCHEMATC

Commit message: ended clavier schematic
Parts:
- removed R_usb (x2): R, symbol R
- added .: AVR-PDI, AVR-ISP-6, symbol AVR-ISP-6
Connections:
- wire segments 95 -> 72
- no-connect marks 0 -> 2
Other:
- moved on the sheet: Alim, C, Flash_memory, L, LED_maj, LED_num, LED_spé, R_led
