File: clavier/clavier.sch (KiCad schematic (older format))
At the start: 14 parts

Commit message: Clavier with quartz schematic done
Parts:
- added CLK?: TSX3225, symbol TSX3225
- added U?: 74HC238, symbol 74HC238
- J?: symbol USB_A -> USB_A-RESCUE-clavier
Connections:
- wire segments 72 -> 85
Other:
- moved on the sheet: LED_maj, LED_num, LED_spé, R_led
